Commit message: second commit

File: models/Jetbot_v1/gazebo_controllers.xacro (robot description, xacro)
@@ -2,5 +2,5 @@
 <robot xmlns:xacro="http://www.ros.org/wiki/xacro">
 <!-- Gazebo Drive control -->
-	 <!-- <gazebo>
+	 <gazebo>
         <plugin name="diff_drive" filename="libgazebo_ros_diff_drive.so">
 			<ros>
@@ -19,10 +19,9 @@
             <publish_wheel_tf>true</publish_wheel_tf>
         </plugin>
-    </gazebo> -->
+    </gazebo>
 <!-- Gazebo Lidar control -->
     <gazebo reference="laser_frame">
         <material>Gazebo/Black</material>
         <sensor name="laser" type="ray">
-            <pose> 0 0 0 0 0 0 </pose>
             <visualize>false</visualize>
             <update_rate>10</update_rate>
@@ -36,5 +35,5 @@
                 </scan>
                 <range>
-                    <min>0.11</min>
+                    <min>0.08</min>
                     <max>10</max>
                 </range>

File: models/Jetbot_v1/lidar.xacro (robot description, xacro)
@@ -5,12 +5,12 @@
         <parent link="chassis"/>
         <child link="laser_frame"/>
-        <origin xyz="0.0 0.0 0.10685" rpy=" 0 0 0 "/>
+        <origin xyz="0.0 0.0 0.11935" rpy=" 0 0 0 "/>
     </joint>
     <link name="laser_frame">
         <xacro:inertial_cylinder mass="0.01" radius="0.0325" length="0.027">
-			<origin xyz="0.0 0.0 0.0135" rpy="0 0 0"/>
+			<origin xyz="0.0 0.0 0.0" rpy="0 0 0"/>
 		</xacro:inertial_cylinder>
     	<visual>
-			<origin xyz="0.0 0.0 0.0135" rpy="0 0 0"/>
+			<origin xyz="0.0 0.0 0.0" rpy="0 0 0"/>
   			<geometry>
   				<cylinder radius="0.0325" length="0.027"/>
@@ -19,5 +19,5 @@
 		</visual>
 		<collision>
-			<origin xyz="0.0 0.0 0.0135" rpy="0 0 0"/>
+			<origin xyz="0.0 0.0 0.0" rpy="0 0 0"/>
   			<geometry>
   				<cylinder radius="0.0325" length="0.027"/>

File: models/Jetbot_v1/model.urdf.xacro (robot description, xacro)
@@ -102,5 +102,5 @@
 		<collision>
   			<geometry>
-  				<cylinder radius="0.0325" length="0.027"/>
+  				<sphere radius="0.0325"/>
   			</geometry>
 		</collision>
@@ -130,5 +130,5 @@
 		<collision>
   			<geometry>
-  				<cylinder radius="0.0325" length="0.027"/>
+  				<sphere radius="0.0325"/>
   			</geometry>
 		</collision>
