Commit message: slam implementation

File: models/Jetbot_v1/camera.xacro (robot description, xacro)
@@ -2,11 +2,11 @@
 <robot xmlns:xacro="http://www.ros.org/wiki/xacro">
 <!--Camera-->
-	<joint name="camera_joint" type="fixed">
+	<joint name="${robot_name}/camera_joint" type="fixed">
     	<origin xyz="0.10315 0.0 0.06" rpy="0 0.1 0"/>
-    	<parent link="chassis"/>
-    	<child link="camera_link"/>
+    	<parent link="${robot_name}/chassis"/>
+    	<child link="${robot_name}/camera_link"/>
     </joint>
 z
-    <link name="camera_link">
+    <link name="${robot_name}/camera_link">
 		<xacro:inertial_box mass="0.05" x="0.01" y="0.02" z="0.02">
 			<origin xyz="0.0 0.0 0.0" rpy="0 0 0"/>

File: models/Jetbot_v1/gazebo_controllers.xacro (robot description, xacro)
@@ -7,12 +7,12 @@
 				<namespace>${robot_name}</namespace>
             </ros>
-            <left_joint>leftWheel_joint</left_joint>
-            <right_joint>rightWheel_joint</right_joint>
+            <left_joint>${robot_name}/leftWheel_joint</left_joint>
+            <right_joint>${robot_name}/rightWheel_joint</right_joint>
             <wheel_separation>0.1863</wheel_separation>
             <wheel_diameter>0.065</wheel_diameter>
             <max_wheel_torque>200</max_wheel_torque>
             <max_wheel_acceleration>10.0</max_wheel_acceleration>
-            <odometry_frame>odom</odometry_frame>
-            <robot_base_frame>base_link</robot_base_frame>
+            <odometry_frame>${robot_name}/odom</odometry_frame>
+            <robot_base_frame>${robot_name}/base_link</robot_base_frame>
             <publish_odom>true</publish_odom>
             <publish_odom_tf>true</publish_odom_tf>
@@ -21,5 +21,5 @@
     </gazebo>
 <!-- Gazebo Lidar control -->
-    <gazebo reference="laser_frame">
+    <gazebo reference="${robot_name}/laser_frame">
         <material>Gazebo/Black</material>
         <sensor name="laser" type="ray">
@@ -45,10 +45,10 @@
                 </ros>
                 <output_type>sensor_msgs/LaserScan</output_type>
-                <frame_name>laser_frame</frame_name>
+                <frame_name>${robot_name}/laser_frame</frame_name>
             </plugin>
         </sensor>
     </gazebo>
 <!-- Gazebo Camera control -->
- 	<gazebo reference="camera_link">
+ 	<gazebo reference="${robot_name}/camera_link">
         <material>Gazebo/Black</material>
         <sensor name="camera" type="camera">
@@ -68,5 +68,5 @@
             </camera>
             <plugin name="camera_controller" filename="libgazebo_ros_camera.so">
-                <frame_name>camera_link</frame_name>
+                <frame_name>${robot_name}/camera_link</frame_name>
 				<ros>
 					<namespace>${robot_name}</namespace>

File: models/Jetbot_v1/lidar.xacro (robot description, xacro)
@@ -2,10 +2,10 @@
 <robot xmlns:xacro="http://www.ros.org/wiki/xacro">
     <!--Lidar-->
-	<joint name="laser_joint" type="fixed">
-        <parent link="chassis"/>
-        <child link="laser_frame"/>
+	<joint name="${robot_name}/laser_joint" type="fixed">
+        <parent link="${robot_name}/chassis"/>
+        <child link="${robot_name}/laser_frame"/>
         <origin xyz="0.0 0.0 0.11935" rpy=" 0 0 0 "/>
     </joint>
-    <link name="laser_frame">
+    <link name="${robot_name}/laser_frame">
         <xacro:inertial_cylinder mass="0.01" radius="0.0325" length="0.027">
 			<origin xyz="0.0 0.0 0.0" rpy="0 0 0"/>

File: models/Jetbot_v1/model.urdf.xacro (robot description, xacro)
@@ -17,12 +17,12 @@
 		<color rgba="0 1 0 1"/>
 	</material>
-	<link name="base_link"></link>
-<!--Chassis-->
-	<joint name="chassis_joint" type="fixed">
+	<link name="${robot_name}/base_link"></link>
+<!--Chassis"-->
+	<joint name="${robot_name}/chassis_joint" type="fixed">
   		<origin xyz="0.0 0.0 0.0325" rpy="0 0 0"/>
-  		<parent link="base_link"/>
-  		<child link="chassis"/>
+  		<parent link="${robot_name}/base_link"/>
+  		<child link="${robot_name}/chassis"/>
 	</joint>
-    <link name='chassis'>
+    <link name='${robot_name}/chassis'>
 		<xacro:inertial_cylinder mass="2.8943" radius="0.106625" length="0.01">
 			<origin xyz="0.0 0.0 0.015" rpy="0 0 0"/>
@@ -80,15 +80,15 @@
 		</visual>
 	</link>
-	<gazebo reference="chassis">
+	<gazebo reference="${robot_name}/chassis">
 		<material>Gazebo/Green</material>
 	</gazebo>
 <!--Left Wheel-->
-	<joint name="leftWheel_joint" type="continuous">
-  		<parent link="chassis"/>
-  		<child link="leftWheel"/>
+	<joint name="${robot_name}/leftWheel_joint" type="continuous">
+  		<parent link="${robot_name}/chassis"/>
+  		<child link="${robot_name}/leftWheel"/>
 		<origin xyz="0.0 0.09315 0.0" rpy="-1.5707 0 0"/>
 		<axis xyz="0 0 1"/>
 	</joint>
-    <link name='leftWheel'>
+    <link name='${robot_name}/leftWheel'>
 		<xacro:inertial_cylinder mass="0.031" radius="0.0325" length="0.027">
 			<origin xyz="0 0 0" rpy="0 0 0"/>
@@ -106,5 +106,5 @@
 		</collision>
 	</link>
-	<gazebo reference="leftWheel">
+	<gazebo reference="${robot_name}/leftWheel">
 		<material>Gazebo/Blue</material>
 		<mu1 value="1.0"/>
@@ -112,11 +112,11 @@
 	</gazebo>
 <!--Right Wheel-->
-	<joint name="rightWheel_joint" type="continuous">
-  		<parent link="chassis"/>
-  		<child link="rightWheel"/>
+	<joint name="${robot_name}/rightWheel_joint" type="continuous">
+  		<parent link="${robot_name}/chassis"/>
+  		<child link="${robot_name}/rightWheel"/>
 		<origin xyz="0.0 -0.09315 0.0" rpy="1.5707 0 0"/>
 		<axis xyz="0 0 -1"/>
 	</joint>
-    <link name='rightWheel'>
+    <link name='${robot_name}/rightWheel'>
 		<xacro:inertial_cylinder mass="0.031" radius="0.0325" length="0.027">
 			<origin xyz="0 0 0" rpy="0 0 0"/>
@@ -134,5 +134,5 @@
 		</collision>
 	</link>
-	<gazebo reference="rightWheel">
+	<gazebo reference="${robot_name}/rightWheel">
 		<material>Gazebo/Blue</material>
 		<mu1 value="1.0"/>
@@ -140,10 +140,10 @@
 	</gazebo>
 <!--Front Caster-->
-	<joint name="frontCaster_joint" type="fixed">
-  		<parent link="chassis"/>
-  		<child link="frontCaster"/>
+	<joint name="${robot_name}/frontCaster_joint" type="fixed">
+  		<parent link="${robot_name}/chassis"/>
+  		<child link="${robot_name}/frontCaster"/>
 		<origin xyz="0.09315 0.0 0.0" rpy="0 0 0"/>
 	</joint>
-    <link name='frontCaster'>
+    <link name='${robot_name}/frontCaster'>
 		<xacro:inertial_sphere mass="0.022" radius="0.022">
 			<origin xyz="0 0 -0.01" rpy="0 0 0"/>
@@ -163,5 +163,5 @@
 		</collision>
 	</link>
-	<gazebo reference="frontCaster">
+	<gazebo reference="${robot_name}/frontCaster">
 		<material>Gazebo/Black</material>
 		<mu1 value="0.01"/>
@@ -169,10 +169,10 @@
 	</gazebo>
 <!--Rear Caster-->
-	<joint name="rearCaster_joint" type="fixed">
-  		<parent link="chassis"/>
-  		<child link="rearCaster"/>
+	<joint name="${robot_name}/rearCaster_joint" type="fixed">
+  		<parent link="${robot_name}/chassis"/>
+  		<child link="${robot_name}/rearCaster"/>
 		<origin xyz="-0.09315 0.0 0.0" rpy="0 0 0"/>
 	</joint>
-    <link name='rearCaster'>
+    <link name='${robot_name}/rearCaster'>
 		<xacro:inertial_sphere mass="0.022" radius="0.022">
 			<origin xyz="0 0 -0.01" rpy="0 0 0"/>
@@ -192,5 +192,5 @@
 		</collision>
 	</link>
-	<gazebo reference="rearCaster">
+	<gazebo reference="${robot_name}/rearCaster">
 		<material>Gazebo/Black</material>
 		<mu1 value="0.01"/>
